Commit message: Add namespace for gazebo_ros in xacro files

File: irobot_create_common/irobot_create_description/urdf/bumper.urdf.xacro (robot description, xacro)
@@ -51,5 +51,5 @@
         <plugin name="${name}_plugin" filename="libgazebo_ros_create_bumper.so">
           <ros>
-            <namespace>$(arg namespace)</namespace>
+            <namespace>/$(arg namespace)</namespace>
             <remapping>~/out:=_internal/bumper/event</remapping>
           </ros>

File: irobot_create_common/irobot_create_description/urdf/create3.urdf.xacro (robot description, xacro)
@@ -43,5 +43,5 @@
   <xacro:property name="base_link_z_offset"     value="${6.42*cm2m}"/>
   <!-- Docking properties -->
-  <xacro:property name="robot_model_name" value="create3"/>
+  <xacro:property name="robot_model_name" value="$(arg namespace)"/>
   <xacro:property name="receiver_link_name" value="ir_omni"/>
   <xacro:property name="dock_model_name" value="standard_dock"/>
@@ -102,8 +102,8 @@
     <gazebo>
       <plugin name="gazebo_ros2_control" filename="libgazebo_ros2_control.so">
+        <ros>
+          <namespace>/$(arg namespace)</namespace>
+        </ros>
         <parameters> $(find irobot_create_control)/config/$(arg namespace).yaml </parameters>
-        <ros>
-          <namespace>$(arg namespace)</namespace>
-        </ros>
       </plugin>
     </gazebo>
@@ -209,5 +209,5 @@
       <plugin name="gazebo_ros_p3d_robot" filename="libgazebo_ros_p3d.so">
         <ros>
-          <namespace>$(arg namespace)</namespace>
+          <namespace>/$(arg namespace)</namespace>
           <remapping>odom:=sim_ground_truth_pose</remapping>
         </ros>
@@ -224,5 +224,5 @@
       <plugin name="dock_status_publisher" filename="libgazebo_ros_create_docking_status.so">
         <ros>
-          <namespace>$(arg namespace)</namespace>
+          <namespace>/$(arg namespace)</namespace>
           <remapping>~/out:=dock</remapping>
         </ros>

File: irobot_create_common/irobot_create_description/urdf/sensors/cliff_sensor.urdf.xacro (robot description, xacro)
@@ -27,5 +27,5 @@
       <plugin name="${sensor_name}" filename="libgazebo_ros_create_cliff_sensor.so">
         <ros>
-          <namespace>$(arg namespace)</namespace>
+          <namespace>/$(arg namespace)</namespace>
           <remapping>~/out:=_internal/${sensor_name}/event</remapping>
         </ros>

File: irobot_create_common/irobot_create_description/urdf/sensors/imu.urdf.xacro (robot description, xacro)
@@ -59,5 +59,5 @@
         <plugin name="${name}_plugin" filename="libgazebo_ros_create_imu.so">
           <ros>
-            <namespace>$(arg namespace)</namespace>
+            <namespace>/$(arg namespace)</namespace>
             <remapping>~/out:=imu</remapping>
           </ros>

File: irobot_create_common/irobot_create_description/urdf/sensors/ir_intensity.urdf.xacro (robot description, xacro)
@@ -27,5 +27,5 @@
           <plugin filename="libgazebo_ros_create_ir_intensity_sensor.so" name="${link_name}">
             <ros>
-              <namespace>$(arg namespace)</namespace>
+              <namespace>/$(arg namespace)</namespace>
               <remapping>~/out:=_internal/${link_name}</remapping>
             </ros>

File: irobot_create_common/irobot_create_description/urdf/sensors/ir_opcode_receivers.urdf.xacro (robot description, xacro)
@@ -52,5 +52,5 @@
         <plugin name="${name}_plugin" filename="libgazebo_ros_create_ir_opcode.so">
           <ros>
-            <namespace>$(arg namespace)</namespace>
+            <namespace>/$(arg namespace)</namespace>
             <remapping>~/out:=ir_opcode</remapping>
           </ros>

File: irobot_create_common/irobot_create_description/urdf/wheel_drop.urdf.xacro (robot description, xacro)
@@ -44,5 +44,5 @@
       <plugin name="${wd_link_name}_plugin" filename="libgazebo_ros_create_wheel_drop.so">
         <ros>
-          <namespace>$(arg namespace)</namespace>
+          <namespace>/$(arg namespace)</namespace>
           <remapping>~/out:=_internal/wheel_drop/${name}_wheel/event</remapping>
         </ros>
